Commit message: Fix lidar model inclusion and update caster wheel joint definitions in scuttle_ydlidar.xacro

File: platform/scuttle/ROS2/src/generic_robot_driver/urdf/scuttle_ydlidar.xacro (robot description, xacro)
@@ -4,10 +4,10 @@
   <xacro:include filename="$(find generic_robot_driver)/urdf/materials.xacro" />
   <xacro:include filename="$(find generic_robot_driver)/urdf/scuttle.trans" />
-  <!-- <xacro:include filename="$(find generic_robot_driver)/urdf/scuttle.gazebo" /> -->
+  <xacro:include filename="$(find generic_robot_driver)/urdf/scuttle.gazebo" />
   <!-- <xacro:include filename="$(find realsense2_description)/urdf/_d435i.urdf.xacro"/> -->
   <link name="base_footprint"></link>
   <link name="base_link">
     <inertial>
-      <origin rpy="0 0 0" xyz="2.12433370053547e-05 -0.07877992189559235 0.07392564365565002" />
+      <origin rpy="0 0 0" xyz="0.12 0 0" />
       <mass value="3.288323846275119" />
       <inertia ixx="0.038876" ixy="1.3e-05" ixz="1e-06" iyy="0.047513" iyz="0.000486" izz="0.084083" />
@@ -215,5 +215,5 @@
     <axis xyz="0.0 -0.0 1.0" />
   </joint>
-  <joint name="r_caster_wheel_joint" type="continuous">
+  <joint name="l_caster_wheel_joint" type="continuous">
     <origin rpy="0 0 0" xyz="-0.017792 0.024 -0.034" />
     <parent link="l_caster_swivel_1" />
@@ -221,5 +221,5 @@
     <axis xyz="1.0 0.0 -0.0" />
   </joint>
-  <joint name="l_caster_wheel_joint" type="continuous">
+  <joint name="r_caster_wheel_joint" type="continuous">
     <origin rpy="0 0 0" xyz="0.014208 0.024 -0.034" />
     <parent link="r_caster_swivel_1" />

Commit message: Update cartographer.launch.py to set use_sim_time to false; modify scuttle_ydlidar.xacro to include D435i sensor and adjust lidar joint origin

File: platform/scuttle/ROS2/src/generic_robot_driver/urdf/scuttle_ydlidar.xacro (robot description, xacro)
@@ -5,5 +5,5 @@
   <xacro:include filename="$(find generic_robot_driver)/urdf/scuttle.trans" />
   <xacro:include filename="$(find generic_robot_driver)/urdf/scuttle.gazebo" />
-  <!-- <xacro:include filename="$(find realsense2_description)/urdf/_d435i.urdf.xacro"/> -->
+  <xacro:include filename="$(find realsense2_description)/urdf/_d435i.urdf.xacro"/>
   <link name="base_footprint"></link>
   <link name="base_link">
@@ -199,5 +199,5 @@
   </joint>
   <joint name="lidar" type="fixed">
-    <origin rpy="0 0 0" xyz="0.2125 0.0 0.40" />
+    <origin rpy="0 0 0" xyz="0.15 0.0 0.43" />
     <parent link="base_link" />
     <child link="lidar_1" />
@@ -227,7 +227,7 @@
     <axis xyz="-1.0 -0.0 0.0" />
   </joint>
-  <!-- <xacro:sensor_d435i parent="base_link" use_nominal_extrinsics="$(arg
+  <xacro:sensor_d435i parent="base_link" use_nominal_extrinsics="$(arg
   use_nominal_extrinsics)">
     <origin rpy="0 0 0" xyz="0.25 0 0.28" />
-</xacro:sensor_d435i> -->
+</xacro:sensor_d435i>
 </robot>

Commit message: changes

File: platform/scuttle/ROS2/src/generic_robot_driver/urdf/scuttle_ydlidar.xacro (robot description, xacro)
@@ -5,5 +5,5 @@
   <xacro:include filename="$(find generic_robot_driver)/urdf/scuttle.trans" />
   <xacro:include filename="$(find generic_robot_driver)/urdf/scuttle.gazebo" />
-  <xacro:include filename="$(find realsense2_description)/urdf/_d435i.urdf.xacro"/>
+  <xacro:include filename="$(find realsense2_description)/urdf/_d435i.urdf.xacro" />
   <link name="base_footprint"></link>
   <link name="base_link">
@@ -208,4 +208,5 @@
     <child link="r_caster_swivel_1" />
     <axis xyz="0.0 0.0 1.0" />
+    <dynamics damping="0.01" friction="0.1"/>
   </joint>
   <joint name="l_caster_swivel_joint" type="continuous">
@@ -214,4 +215,5 @@
     <child link="l_caster_swivel_1" />
     <axis xyz="0.0 -0.0 1.0" />
+    <dynamics damping="0.01" friction="0.1"/>
   </joint>
   <joint name="l_caster_wheel_joint" type="continuous">
@@ -230,4 +232,4 @@
   use_nominal_extrinsics)">
     <origin rpy="0 0 0" xyz="0.25 0 0.28" />
-</xacro:sensor_d435i>
+  </xacro:sensor_d435i>
 </robot>
